File: kicad/mdb-slave-esp32s3/mdb-slave-esp32s3.kicad_pcb (KiCad board)
At the start: 2 copper layers, 39 x 40 mm, 46 parts, among them J1 MDB_Connector, J2 USB_C_Receptacle_USB2.0_16P, J3 Conn_01x03_Pin, J8 Conn_01x04_Pin, Q7 MMBT3904, SW1 SW_Push, U1 TLP785, U3 ESP32-S3FH4R2, U4 TLP785, U5 LM2594HVM-3.3, Y1 Crystal_GND24

Commit message: feat(kicad-slave): add 2x11 extension pin header (J4) for add-on modules
Reproduces the historical breakout header (commit c5da6d6) on the WiFi
ESP32-S3 slave so extension modules can be plugged on top. J4 =
Conn_02x11_Odd_Even with the exact historical pin->net mapping: UART0
(u0txd/u0rxd) + all 16 GPIOs (io1..io21) + 3V3 + VIN + 3x GND.

- Schematic: J4 + 22 net labels, pinout verified pin-by-pin vs c5da6d6
- PCB: left Edge.Cuts extended 9.5mm (board 48.5x40mm); J4 placed in the
  new strip, all 22 pads net-assigned, clears the H1 mounting hole
- schematic<->PCB net-consistent (22/22); DRC adds zero new violations
  vs baseline (and removed 4 pre-existing copper_edge_clearance errors)
- J3/J8/SW1/H1 and all other parts unchanged
- Routing pending (traces not yet drawn)

Spec: docs/superpowers/specs/2026-06-08-slave-extension-header-design.md

Co-Authored-By: Claude Opus 4.8 <noreply@anthropic.com>
Parts:
- added J4: Conn_02x11_Odd_Even, Connector_PinHeader_2.54mm:PinHeader_2x11_P2.54mm_Vertical, F.Cu at (161.0, 91.2)
Other:
- board size 39 x 40 mm -> 48.5 x 40 mm
