File: kicad/mdb_slave_esp32s3-wroom-u1/mdb_slave_esp32s3-wroom-u1.kicad_sch (KiCad schematic)
At the start: 65 parts, among them J1 USB_C_Receptacle_USB2.0_16P, J10 Conn_01x04_Pin_JST, J11 Screw_Terminal_01x03, J12 MDB_Connector, J13 Screw_Terminal_01x03, J14 Screw_Terminal_01x03, J2 Screw_Terminal_01x02, J3 Screw_Terminal_01x02, J4 Screw_Terminal_01x03, J5 Screw_Terminal_01x03, J6 Screw_Terminal_01x03, J7 Conn_01x06_Pin, J8 Conn_01x03_Pin_JST, J9 Conn_01x04_Pin, Q1 MMBT3904, Q2 MMBT3904, Q3 MMBT3904, SW1 SW_Push, U1 ESP32-S3-WROOM-1U-N16R2, U2 AP63203QWU-7, U3 TLP785, U4 TLP785

Commit message: Update footprint and symbol for BUZZER + ESP32S3-WROOM-U1. PCB empty with all component on side.
Parts:
- removed BZ1: Buzzer, ProtoFlow.pretty:BUZ-TH_BD23.0-P15.00-D0.8-FD, symbol Device:Buzzer
- added BUZZER1: MLT-8530, easyeda2kicad:BUZ-SMD_4P-L8.5-W8.5-P8.50-BR, symbol easyeda2kicad:MLT-8530
- C1, C2, L1, R1, R10, R11, R12, R13, R14, R15, R16, R17, R18, R19, R2, R20, R21, R22, R3, R4, R5, R6, R7, R8, R9: footprint ProtoFlow.pretty:LED0603-RD -> (none); Protoflow_Source kicad -> (none)
- C3: footprint ProtoFlow.pretty:CONN-TH_B4B-PH-K-S -> Capacitor_SMD:C_0603_1608Metric; Attrition Qty (none) -> 10; Capacitance (none) -> 10nF; Category (none) -> Capacitors,Multilayer Ceramic Capacitors MLCC - SMD/SMT; Class (none) -> Basic Component; LCSC (none) -> C57112; Manufacturer (none) -> FH(Guangdong Fenghua Advanced Tech); Minimum Qty (none) -> 20; Part (none) -> 0603B103K500NT; Price (none) -> 0.005USD; Process (none) -> SMT; Protoflow_Source kicad -> (none); Stock (none) -> 5921160; Temperature Coefficient (none) -> X7R; Tolerance (none) -> ±10%; Voltage Rated (none) -> 50V
- C4: footprint ProtoFlow.pretty:CONN-TH_B4B-PH-K-S -> Capacitor_SMD:C_0603_1608Metric; Attrition Qty (none) -> 10; Capacitance (none) -> 100nF; Category (none) -> Capacitors,Multilayer Ceramic Capacitors MLCC - SMD/SMT; Class (none) -> Basic Component; LCSC (none) -> C14663; Manufacturer (none) -> YAGEO; Minimum Qty (none) -> 20; Part (none) -> CC0603KRX7R9BB104; Price (none) -> 0.006USD; Process (none) -> SMT; Protoflow_Source kicad -> (none); Stock (none) -> 70324515; Temperature Coefficient (none) -> X7R; Tolerance (none) -> ±10%; Voltage Rated (none) -> 50V
- C5, C6: footprint ProtoFlow.pretty:CONN-TH_B4B-PH-K-S -> Capacitor_SMD:C_0603_1608Metric; Attrition Qty (none) -> 10; Capacitance (none) -> 220nF; Category (none) -> Capacitors,Multilayer Ceramic Capacitors MLCC - SMD/SMT; Class (none) -> Basic Component; LCSC (none) -> C21120; Manufacturer (none) -> Samsung Electro-Mechanics; Minimum Qty (none) -> 20; Part (none) -> CL10B224KA8NNNC; Price (none) -> 0.009USD; Process (none) -> SMT; Protoflow_Source kicad -> (none); Stock (none) -> 781839; Temperature Coefficient (none) -> X7R; Tolerance (none) -> ±10%; Voltage Rated (none) -> 25V
- D1: footprint ProtoFlow.pretty:DO-41_BD2.4-L4.7-P8.70-D0.9-RD -> (none); Protoflow_Source kicad -> (none)
- D2: footprint ProtoFlow.pretty:CONN-TH_B4B-PH-K-S -> LED_SMD:LED_WS2812B-2020_PLCC4_2.0x2.0mm; Protoflow_Source kicad -> (none)
- D3, D4: footprint ProtoFlow.pretty:DFN1006-2L-RD -> (none); Protoflow_Source kicad -> (none)
- D5, D6: footprint ProtoFlow.pretty:SOD-323_L1.8-W1.3-LS2.5-RD -> Diode_SMD:D_SOD-323; Protoflow_Source kicad -> (none)
- F1, J1, J10, J11, J12, J13, J14, J2, J3, J4, J5, J6, J7, J8, J9, SW1, TH1: footprint ProtoFlow.pretty:CONN-TH_B4B-PH-K-S -> (none); Protoflow_Source kicad -> (none)
- H1, H2, H3, H4, H5: footprint ProtoFlow.pretty:CONN-TH_B4B-PH-K-S -> (none); Protoflow_Source kicad -> (none); now left out of the parts list
- Q1, Q2, Q3: footprint ProtoFlow.pretty:SOT-23-3_L2.9-W1.3-P1.90-LS2.4-BR -> Package_TO_SOT_SMD:SOT-23; Protoflow_Source kicad -> (none)
- U1: footprint ProtoFlow.pretty:WIRELM-SMD_ESP32-S3-WROOM-1U -> RF_Module:ESP32-S3-WROOM-1U; Protoflow_Source kicad -> (none)
- U2: footprint ProtoFlow.pretty:TSOT-26_L2.9-W1.6-P0.95-LS2.8-BL -> Package_TO_SOT_SMD:TSOT-23-6; Protoflow_Source kicad -> (none)
- U3, U4: footprint ProtoFlow.pretty:DIP-4_L6.4-W4.6-P2.54-LS7.6-BL -> Package_DIP:DIP-4_W7.62mm; Protoflow_Source kicad -> (none)
Connections:
- net GND: now also BUZZER1.2
- net io10: now also J10.3 (Pin_3), R16.1
- net io11: now also J10.4 (Pin_4), R15.1
- net io7: now also R7.1, TH1.2
- net at R12.1: now also BUZZER1.1 (+)
Other:
- company: Protoflow -> (none)
- title: Untitled -> (none)

Commit message: Move custom_input2/3 from IO8/IO9 to IO47/IO48
IO8/IO9 collided with PIN_DEX_RX/PIN_DEX_TX on the original
mdb-slave-esp32s3 board, so flashing the wrong firmware onto either
board would silently misdrive these pins instead of erroring.

IO17/IO18 were considered as an alternative but rejected — those
collide with PIN_SIM7080G_TX/RX on the basic-plus/cellular variant
instead, trading one cross-board conflict for another.

IO47/IO48 are free on every board variant and unaffected by
Quad-vs-Octal PSRAM pin reservations (unlike IO35-37), so J13/J14 and
their pull-up resistors are rerouted there. IO8/IO9 are now
no-connect.

Firmware side already updated on feature/esp32s3-wroom-u1-firmware
(PIN_CUSTOM_INPUT1/2/3 defines).
Connections:
- net io47: now reaches U1.24 (IO47)
- net io47: now also J13.3 (Pin_3), R19.1
- net io48: now reaches U1.25 (IO48)
- net io48: now also J14.3 (Pin_3), R22.1
- removed net io8: J13.3 (Pin_3), R19.1, U1.12 (IO8)
- removed net io9: J14.3 (Pin_3), R22.1, U1.17 (IO9)
Changed lines of the file:
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@@
 		)
 	)
-	(text_box "io1    ->  relay1\nio2    ->  relay2\nio3    (free)\nio4    ->  mdb/rx\nio5    ->  mdb/tx\nio6    ->  custom_input1\nio7    ->  thermistor\nio8    ->  custom_input2\nio9    ->  custom_input3\nio10   ->  i2c/sda\nio11   ->  i2c/scl\nio12   ->  buzzer\nio13   ->  pulse\nio14   (free)\nio15   ->  1wire/bus1\nio16   ->  1wire/bus2\nio17   (free)\nio18   (free)\nio21   ->  led\n\nu0txd/u0rxd  ->  uart_debug\nio39   ->  jtag/tck\nio40   ->  jtag/tdo\nio41   ->  jtag/tdi\nio42   ->  jtag/tms\n\nio35, io36, io37, io38, io47, io48 (free)"
+	(text_box "io1    ->  relay1\nio2    ->  relay2\nio3    (free)\nio4    ->  mdb/rx\nio5    ->  mdb/tx\nio6    ->  custom_input1\nio7    ->  thermistor\nio8    ->  free (to avoid conflict with old PCB)\nio9    ->  free (to avoid conflict with old PCB)\nio10   ->  i2c/sda\nio11   ->  i2c/scl\nio12   ->  buzzer\nio13   ->  pulse\nio14   (free)\nio15   ->  1wire/bus1\nio16   ->  1wire/bus2\nio17   (free)\nio18   (free)\nio21   ->  led\n\nio35, io36, io37, io38 (free)\n\nu0txd/u0rxd  ->  uart_debug\nio39   ->  jtag/tck\nio40   ->  jtag/tdo\nio41   ->  jtag/tdi\nio42   ->  jtag/tms\n\nio47    ->  custom_input2\nio48    ->  custom_input3"
 		(exclude_from_sim no)
-		(at 256.54 223.52 0)
-		(size 41.91 59.1533)
+		(at 247.65 215.8782 0)
+		(size 50.8 67.3318)
 		(margins 0.9525 0.9525 0.9525 0.9525)
 		(stroke
@@
 	)
 	(no_connect
+		(at 93.98 107.95)
+	)
+	(no_connect
 		(at 347.98 45.72)
 	)
@@
 	)
 	(no_connect
-		(at 124.46 125.73)
-	)
-	(no_connect
 		(at 124.46 237.49)
 	)
@@
 	)
 	(no_connect
+		(at 93.98 105.41)
+	)
+	(no_connect
 		(at 93.98 120.65)
-	)
-	(no_connect
-		(at 124.46 123.19)
 	)
 	(no_connect
@@
 	(wire
 		(pts
+			(xy 124.46 125.73) (xy 128.27 125.73)
+		)
+		(stroke
+			(width 0)
+			(type default)
+		)
+	)
+	(wire
+		(pts
 			(xy 66.04 73.66) (xy 67.31 73.66)
 		)
@@
 	(wire
 		(pts
-			(xy 87.63 107.95) (xy 93.98 107.95)
-		)
-		(stroke
-			(width 0)
-			(type default)
-		)
-	)
-	(wire
-		(pts
 			(xy 377.19 138.43) (xy 373.38 138.43)
 		)
@@
 	(wire
 		(pts
-			(xy 87.63 105.41) (xy 93.98 105.41)
-		)
-		(stroke
-			(width 0)
-			(type default)
-		)
-	)
-	(wire
-		(pts
 			(xy 229.87 49.53) (xy 229.87 57.15)
 		)
@@
 		(pts
 			(xy 285.75 81.28) (xy 278.13 81.28)
+		)
+		(stroke
+			(width 0)
+			(type default)
+		)
+	)
+	(wire
+		(pts
+			(xy 124.46 123.19) (xy 128.27 123.19)
 		)
 		(stroke
@@
 		)
 	)
-	(label "io9"
-		(at 87.63 107.95 180)
-		(effects
-			(font
-				(size 1.27 1.27)
-			)
-			(justify right bottom)
-		)
-	)
 	(label "vin"
 		(at 124.46 185.42 180)
@@
 		)
 	)
-	(label "io8"
+	(label "io47"
 		(at 360.68 143.51 0)
 		(effects
@@
 		)
 	)
+	(label "io47"
+		(at 128.27 123.19 0)
+		(effects
+			(font
+				(size 1.27 1.27)
+			)
+			(justify left bottom)
+		)
+	)
 	(label "mdb_master_receive"
 		(at 363.22 40.64 0)
@@
 		)
 	)
-	(label "io8"
-		(at 87.63 105.41 180)
-		(effects
-			(font
-				(size 1.27 1.27)
-			)
-			(justify right bottom)
-		)
-	)
 	(label "io42"
 		(at 265.43 151.13 0)
@@
 		)
 	)
-	(label "io9"
+	(label "io48"
 		(at 387.35 143.51 0)
 		(effects
@@
 		(effects
 			(font
+				(size 1.27 1.27)
+			)
+			(justify left bottom)
+		)
+	)
+	(label "io48"
+		(at 128.27 125.73 0)
+		(effects
+			(font

Commit message: fix(hardware): add GPIO3 pull-down strap for WROOM-U1 board detection
Add a 10kΩ pull-down resistor from GPIO3 (pin 15 on the ESP32-S3-WROOM-1
symbol) to GND. This was previously unconnected on this board revision.
Lets detect_board_variant() read GPIO3 LOW at boot and correctly identify
the WROOM-U1 board, so DEX/UART1 init is skipped as intended (matches the
firmware-side README in mdb-slave-esp32s3-wroom-u1).
Parts:
- added R23: 10k, Resistor_SMD:R_0603_1608Metric, symbol Device:R
- BUZZER1: LCSC Part C94599 -> (none); LCSC# (none) -> C94599
- C1, C2: footprint (none) -> Capacitor_SMD:C_0603_1608Metric; LCSC# (none) -> C14663
- C3: LCSC C57112 -> (none); LCSC# (none) -> C19702
- C4: LCSC C14663 -> (none); LCSC# (none) -> C14663
- C5, C6: LCSC C21120 -> (none); LCSC# (none) -> C59461
- D1: footprint (none) -> Diode_SMD:D_SOD-123; LCSC# (none) -> C64894
- D2: LCSC# (none) -> C5349957
- D3, D4: footprint (none) -> Diode_SMD:D_SOD-123; LCSC# (none) -> C437999
- D5, D6: LCSC# (none) -> C2128
- F1: footprint (none) -> Fuse:Fuse_1812_4532Metric; LCSC# (none) -> C7542972
- J1: footprint (none) -> Connector_USB:USB_C_Receptacle_G-Switch_GT-USB-7010ASV; LCSC# (none) -> C2988369
- J10: footprint (none) -> Connector_JST:JST_PH_B4B-PH-K_1x04_P2.00mm_Vertical; LCSC# (none) -> C131334
- J11, J13, J14, J4, J5, J6: footprint (none) -> EasyEDA2Kicad:CONN-TH_3P-P2.54_DIBO_DB141R-2.54-3P; LCSC# (none) -> C2898755
- J12: footprint (none) -> Connector_Molex:Molex_Mini-Fit_Jr_5566-06A_2x03_P4.20mm_Vertical; LCSC# (none) -> C2845778
- J2, J3: footprint (none) -> EasyEDA2Kicad:CONN-TH_2P-P2.54_DIBO_DB141R-2.54-2P; LCSC# (none) -> C2898754
- J7: footprint (none) -> Connector_PinHeader_2.54mm:PinHeader_1x06_P2.54mm_Vertical; LCSC# (none) -> C37208
- J8: footprint (none) -> Connector_JST:JST_PH_B3B-PH-K_1x03_P2.00mm_Vertical; LCSC# (none) -> C131339
- J9: footprint (none) -> Connector_PinHeader_2.54mm:PinHeader_1x04_P2.54mm_Vertical; LCSC# (none) -> C124378
- L1: footprint (none) -> Inductor_SMD:L_TechFuse_SL0420; LCSC# (none) -> C22463807
- Q1, Q2, Q3: LCSC# (none) -> C916374
- R1, R17, R19, R2, R22, R5, R6, R7: footprint (none) -> Resistor_SMD:R_0603_1608Metric; LCSC# (none) -> C98220
- R10, R20, R9: footprint (none) -> Resistor_SMD:R_0603_1608Metric; LCSC# (none) -> C2907002
- R11, R13, R14, R15, R16, R8: footprint (none) -> Resistor_SMD:R_0603_1608Metric; LCSC# (none) -> C23162
- R12: footprint (none) -> Resistor_SMD:R_0603_1608Metric; LCSC# (none) -> C2906981
- R18, R21: footprint (none) -> Resistor_SMD:R_0603_1608Metric; LCSC# (none) -> C22356627
- R3, R4: footprint (none) -> Resistor_SMD:R_0603_1608Metric; LCSC# (none) -> C2907044
- SW1: footprint (none) -> Button_Switch_SMD:SW_Tactile_SPST_NO_Straight_CK_PTS636Sx25SMTRLFS; LCSC# (none) -> C42435421
- TH1: footprint (none) -> Resistor_SMD:R_0603_1608Metric; LCSC# (none) -> C13564
- U1: footprint RF_Module:ESP32-S3-WROOM-1U -> EasyEDA2Kicad:WIRELM-SMD_ESP32-S3-WROOM-1U; LCSC# (none) -> C3013945
- U2: LCSC# (none) -> C5248536
- U3, U4: footprint Package_DIP:DIP-4_W7.62mm -> EasyEDA2Kicad:SMD-4_L4.6-W3.7-P2.54-LS7.0-BR; LCSC# (none) -> C128776
Connections:
- net GND: now also R23.1
- net at U1.15 (IO3): now also R23.2
- no-connect marks 14 -> 13
