File: kicad/mdb_slave_esp32s3-wroom-1u/mdb_slave_esp32s3-wroom-1u.kicad_sch (KiCad schematic)
At the start: 66 parts, among them J1 USB_C_Receptacle_USB2.0_16P, J10 Conn_01x04_Pin_JST, J11 Screw_Terminal_01x03, J12 MDB_Connector, J13 Screw_Terminal_01x03, J14 Screw_Terminal_01x03, J2 Screw_Terminal_01x02, J3 Screw_Terminal_01x02, J4 Screw_Terminal_01x03, J5 Screw_Terminal_01x03, J6 Screw_Terminal_01x03, J7 Conn_01x06_Pin, J8 Conn_01x03_Pin_JST, J9 Conn_01x04_Pin, Q1 MMBT3904, Q2 MMBT3904, Q3 MMBT3904, SW1 SW_Push, U1 ESP32-S3-WROOM-1U-N16R2, U2 AP63203QWU-7, U3 TLP785, U4 TLP785

Commit message: feat(wroom-1u): update PCB to rev1.2 (fully routed) and sync README
Board is now fully routed and fabrication-ready. README updated to
reflect rev1.2 status, the current connector reference designators
(J1-J3, P1-P8, H1), and functional blocks, replacing the stale
"not started" rev1.0 content and outdated J1-J14 connector table.
Parts:
- removed BUZZER1: MLT-8530, easyeda2kicad:BUZ-SMD_4P-L8.5-W8.5-P8.50-BR, symbol easyeda2kicad:MLT-8530
- removed C3: 10uF, Capacitor_SMD:C_0603_1608Metric, symbol PCM_JLCPCB-Capacitors:0603,10nF
- removed C4: 100nF, Capacitor_SMD:C_0603_1608Metric, symbol PCM_JLCPCB-Capacitors:0603,100nF
- removed C5, C6: 22uF, Capacitor_SMD:C_0603_1608Metric, symbol PCM_JLCPCB-Capacitors:0603,220nF
- removed D1: Schottky 60V/1A, Diode_SMD:D_SOD-123, symbol Device:D_Schottky
- removed D2: XL-2121RGBC-2812B, LED_SMD:LED_WS2812B-2020_PLCC4_2.0x2.0mm, symbol LED:WS2812B-2020
- removed D4: Schottky 30V/500mA, Diode_SMD:D_SOD-123, symbol Device:D_Schottky
- removed D5, D6: 1N4148WS, Diode_SMD:D_SOD-323, symbol Diode:1N4148WS
- removed F1: 1.1A (33V), Fuse:Fuse_1812_4532Metric, symbol Device:Polyfuse_Small
- removed H1: MountingHole2.5, symbol Mechanical:MountingHole
- removed J1: USB_C_Receptacle_USB2.0_16P, Connector_USB:USB_C_Receptacle_G-Switch_GT-USB-7010ASV, symbol Connector:USB_C_Receptacle_USB2.0_16P
- removed J10: Conn_01x04_Pin_JST, Connector_JST:JST_PH_B4B-PH-K_1x04_P2.00mm_Vertical, symbol Connector:Conn_01x04_Pin
- removed J11, J13, J14, J4, J5, J6: Screw_Terminal_01x03, EasyEDA2Kicad:CONN-TH_3P-P2.54_DIBO_DB141R-2.54-3P, symbol Connector:Screw_Terminal_01x03
- removed J12: MDB_Connector, Connector_Molex:Molex_Mini-Fit_Jr_5566-06A_2x03_P4.20mm_Vertical, symbol Connector_Generic:Conn_02x03_Top_Bottom
- removed J2, J3: Screw_Terminal_01x02, EasyEDA2Kicad:CONN-TH_2P-P2.54_DIBO_DB141R-2.54-2P, symbol Connector:Screw_Terminal_01x02
- removed J7: Conn_01x06_Pin, Connector_PinHeader_2.54mm:PinHeader_1x06_P2.54mm_Vertical, symbol Connector:Conn_01x06_Pin
- removed J8: Conn_01x03_Pin_JST, Connector_JST:JST_PH_B3B-PH-K_1x03_P2.00mm_Vertical, symbol Connector:Conn_01x03_Pin
- removed J9: Conn_01x04_Pin, Connector_PinHeader_2.54mm:PinHeader_1x04_P2.54mm_Vertical, symbol Connector:Conn_01x04_Pin
- removed R23, R5, R6: 10k, Resistor_SMD:R_0603_1608Metric, symbol Device:R
- removed SW1: SW_Push, Button_Switch_SMD:SW_Tactile_SPST_NO_Straight_CK_PTS636Sx25SMTRLFS, symbol Switch:SW_Push
- removed U2: AP63203QWU-7, Package_TO_SOT_SMD:TSOT-23-6, symbol Regulator_Switching:AP63203WU
- removed U3, U4: TLP785, EasyEDA2Kicad:SMD-4_L4.6-W3.7-P2.54-LS7.0-BR, symbol Isolator:TLP785
- added B1, B2: Btn1, Global Libraries:KEY-SMD_B3U-1000PM, symbol Switch:SW_Push
- added BUZZER1: MLT-8530, Global Libraries:BUZ-SMD_4P-L8.5-W8.5-P8.50-BR_C94599, symbol globral_library:MLT-8530
- added C10, C3, C6: 10uF, Capacitor_SMD:C_0603_1608Metric, symbol Device:C
- added C11, C12, C4, C5, C7: 100nF, Capacitor_SMD:C_0603_1608Metric, symbol Device:C
- added C8, C9: 22uF, Capacitor_SMD:C_0603_1608Metric, symbol Device:C
- added D1, D2, D4: 1N4148WS, Diode_SMD:D_SOD-323, symbol Diode:1N4148WS
- added D5, D6: BAT760-7, Diode_SMD:D_SOD-323, symbol Device:D_Schottky
- added F2: Polyfuse, Capacitor_SMD:C_1812_4532Metric, symbol Device:Polyfuse
- added H1: HC-5557-2*3AW, Global Libraries:CONN-TH_6P-P4.20-S5.50_5557-2X3AW_C2845788, symbol globral_library:HC-5557-2*3AW
- added H10: Buzzer_OUT, TestPoint:TestPoint_Pad_D1.0mm, symbol Mechanical:MountingHole_Pad
- added H6: +5V, TestPoint:TestPoint_Pad_D1.0mm, symbol Mechanical:MountingHole_Pad
- added H7: +3V3, TestPoint:TestPoint_Pad_D1.0mm, symbol Mechanical:MountingHole_Pad
- added H8: DO, TestPoint:TestPoint_Pad_D1.0mm, symbol Mechanical:MountingHole_Pad
- added H9: Buzzer_IN, TestPoint:TestPoint_Pad_D1.0mm, symbol Mechanical:MountingHole_Pad
- added J1, J2: Conn_01x06_Pin, Connector_PinSocket_2.54mm:PinSocket_1x06_P2.54mm_Vertical, symbol Connector:Conn_01x06_Pin
- added J3: Conn_01x04_Pin, Connector_JST:JST_XH_B4B-XH-A_1x04_P2.50mm_Vertical, symbol Connector:Conn_01x04_Pin
- added LED1: XL-2121RGBC-2812B, Global Libraries:LED-SMD_4P-L2.1-W2.1-BR_XL-2121RGBC-WS2812B_C5349957, symbol globral_library:XL-2121RGBC-WS2812B
- added P1, P2, P3, P4, P5, P6: WJ500V-5.08-3P-14-00A, Global Libraries:CONN-TH_3P-P5.00_WJ500V-5.08-3P_C72334, symbol globral_library:WJ500V-5.08-3P-14-00A
- added P7, P8: WJ500V-5.08-2P-14-00A, Global Libraries:CONN-TH_2P-P5.00_WJ500V-5.08-2P_C8465, symbol globral_library:WJ500V-5.08-2P-14-00A
- added R5, R6: 0R, Resistor_SMD:R_0603_1608Metric_Pad0.98x0.95mm_HandSolder, symbol Device:R_Small
- added U5, U6: TLP785, Global Libraries:SMD-4_L4.6-W6.5-P2.54-LS10.2-BR_C45445, symbol Isolator:TLP785
- added U8: AP63203QWU-7, Package_TO_SOT_SMD:TSOT-23-6, symbol Regulator_Switching:AP63203WU
- added USBC1: TYPE-C-31-M-12, Global Libraries:USB-C_SMD-TYPE-C-31-M-12, symbol ATMEGA328P_MAX17043_Schematic:USB-C
- C1, C2: LCSC (none) -> C14663; LCSC# C14663 -> (none); MFR.Part # (none) -> CC0603KRX7R9BB104
- D3: value Schottky 30V/500mA -> BAT760-7; footprint Diode_SMD:D_SOD-123 -> Diode_SMD:D_SOD-323; LCSC (none) -> C27636120; LCSC# C437999 -> (none); MFR.Part # (none) -> BAT760-7
- H2, H3, H4, H5: value MountingHole2.5 -> MountingHole; footprint (none) -> MountingHole:MountingHole_2.7mm_M2.5_ISO7380
- L1: footprint Inductor_SMD:L_TechFuse_SL0420 -> Inductor_SMD:L_0603_1608Metric; LCSC (none) -> C12589; LCSC# C22463807 -> (none); MFR.Part # (none) -> SDFL1608Q3R3KTF
- Q1, Q2, Q3: LCSC (none) -> C916374; LCSC# C916374 -> (none); MFR.Part # (none) -> MMBT3904
- R1, R17, R2: value 10k -> 10KΩ; LCSC (none) -> C25804; LCSC# C98220 -> (none); MFR.Part # (none) -> 0603WAF1002T5E
- R10, R20: value 1k -> 10KΩ; LCSC (none) -> C25804; LCSC# C2907002 -> (none); MFR.Part # (none) -> 0603WAF1002T5E
- R11, R8: value 4.7k -> 4.7KΩ; LCSC (none) -> C23162; LCSC# C23162 -> (none); MFR.Part # (none) -> 0603WAF4701T5E
- R12: value 100ohm -> 470Ω; LCSC (none) -> C23179; LCSC# C2906981 -> (none); MFR.Part # (none) -> 0603WAF4700T5E
- R13: value 4.7k -> 10KΩ; LCSC (none) -> C25804; LCSC# C23162 -> (none); MFR.Part # (none) -> 0603WAF1002T5E
- R14, R15: value 4.7k -> 1KΩ; LCSC (none) -> C14676; LCSC# C23162 -> (none); MFR.Part # (none) -> RC0603JR-071KL
- R16: value 4.7k -> 470Ω; LCSC (none) -> C23179; LCSC# C23162 -> (none); MFR.Part # (none) -> 0603WAF4700T5E
- R18: value 470ohm -> 10KΩ; LCSC (none) -> C25804; LCSC# C22356627 -> (none); MFR.Part # (none) -> 0603WAF1002T5E
- R19: value 10k -> 1KΩ; LCSC (none) -> C14676; LCSC# C98220 -> (none); MFR.Part # (none) -> RC0603JR-071KL
- R21: value 470ohm -> 5.1KΩ; LCSC (none) -> C23186; LCSC# C22356627 -> (none); MFR.Part # (none) -> 0603WAF5101T5E
- R22: value 10k -> 5.1KΩ; LCSC (none) -> C23186; LCSC# C98220 -> (none); MFR.Part # (none) -> 0603WAF5101T5E
- R3: value 5.1k -> 470Ω; LCSC (none) -> C23179; LCSC# C2907044 -> (none); MFR.Part # (none) -> 0603WAF4700T5E
- R4: value 5.1k -> 4.7KΩ; LCSC (none) -> C23162; LCSC# C2907044 -> (none); MFR.Part # (none) -> 0603WAF4701T5E
- R7: value 10k -> 4.7KΩ; LCSC (none) -> C23162; LCSC# C98220 -> (none); MFR.Part # (none) -> 0603WAF4701T5E
- R9: value 1k -> 4.7KΩ; LCSC (none) -> C23162; LCSC# C2907002 -> (none); MFR.Part # (none) -> 0603WAF4701T5E
- TH1: footprint Resistor_SMD:R_0603_1608Metric -> Capacitor_SMD:C_0603_1608Metric_Pad1.08x0.95mm_HandSolder; LCSC (none) -> C13564; LCSC# C13564 -> (none); MFR.Part # (none) -> NCP18XH103F03RB
- U1: footprint EasyEDA2Kicad:WIRELM-SMD_ESP32-S3-WROOM-1U -> Global Libraries:WIRELM-SMD_ESP32-S3-WROOM-1U_C3013945; LCSC (none) -> C3013945; LCSC# C3013945 -> (none); MFR.Part # (none) -> ESP32-S3-WROOM-1U-N16R2
Connections:
- net +3V3: now also R1.1, R10.1, R14.1, R18.2, R20.2, R4.1, R7.1, R9.2, C12.2, C3.2, C8.2, C9.2, D1.1 (K), D5.1 (K), H7.1, H9.1, J1.6 (Pin_6), J2.6 (Pin_6), J3.2 (Pin_2), LED1.2 (VDD), P1.2, P2.2, P3.2, P4.2, P5.2, P6.2, P7.2, P8.2, R5.1, U8.1 (FB); no longer C1.2, R1.2, R15.2, R19.2, R2.1, R20.1, R21.1, R22.2, R7.2
- net GND: now also C1.2, R2.2, R21.2, R22.2, TH1.2, B1.1, B2.1, C10.2, C11.2, C12.1, C3.1, C4.2, C5.2, C6.2, C8.1, C9.1, H1.2, J1.5 (Pin_5), J2.5 (Pin_5), J3.1 (Pin_1), LED1.4 (GND), P1.1, P2.1, P3.1, P4.1, P5.1, P6.1, U5.3, U8.4 (GND), USBC1.1 (SH), USBC1.2 (SH), USBC1.3 (SH), USBC1.4 (SH), USBC1.A1 (GND), USBC1.A12 (GND), USBC1.B1 (GND), USBC1.B12 (GND); no longer C1.1, R3.2, R4.2, TH1.1
- net mdb_communications_common: now also H1.6, U5.2, U6.3
- net mdb_master_receive: now also H1.4, U6.4
- net mdb_master_transmit: now also R12.1, H1.5; no longer R18.2
- net GPIO17: now reaches R18.1
- net GPIO17: now also U1.10 (IO17), P2.3
- net at D3.2 (A): now also Q2.3 (C), P8.1; no longer Q1.3 (C)
- net at Q1.1 (B): now also R3.2; no longer R9.1
- net at Q2.1 (B): now also R15.1; no longer R10.1
- net at L1.1: now also C7.2, U8.5 (SW)
- net at Q3.1 (B): now also R19.1; no longer R14.2
- net at Q3.3 (C): now also D5.2 (A), P7.1
- net GPIO12: now reaches R3.1
- net GPIO12: now also U1.20 (IO12)
- net at U1.15 (IO3): now also R2.1
- net GPIO18: now reaches U1.11 (IO18)
- net GPIO18: now also R20.1, P3.3
- net EN: now reaches U1.3 (EN)
- net EN: now also C1.1, R1.2, B1.2, C4.1, J1.1 (Pin_1); no longer R2.2
- net boot renamed IO0
- net IO0: now also R10.2, B2.2, C5.1, J1.4 (Pin_4); no longer R1.1
- net io1 renamed GPIO1
- net GPIO1: now also R19.2; no longer R9.2
- net io10: no longer names the net of R16.1
- net io10: now also D4.2 (A); no longer U1.18 (IO10)
- net io11 renamed GPIO11_SCL
- net GPIO11_SCL: now also R9.1, J3.3 (Pin_3); no longer R15.1
- net io12: no longer names the net of R12.2
- net io12: now also D2.2 (A); no longer U1.20 (IO12)
- net io13: no longer names the net of U1.21 (IO13)
- net io13: no longer R14.1
- net io15 renamed GPIO15
- net GPIO15: now also R4.2, P4.3, P6.3; no longer R8.1
- net io16 renamed GPIO16
- net GPIO16: now also R7.2, P5.3; no longer R13.1
- net io2 renamed GPIO2
- net GPIO2: now also R15.2; no longer R10.2
- net io21 renamed GPIO21
- net GPIO21: now also LED1.1 (DIN)
- net io39 renamed MTCk
- net MTCk: now also J2.4 (Pin_4)
- net io4 renamed GPIO4
- net GPIO4: now also R14.2, U5.4; no longer R20.2
- net io40 renamed MTDO
- net MTDO: now also J2.3 (Pin_3)
- net io41 renamed MTDI
- net MTDI: now also J2.2 (Pin_2)
- net io42 renamed MTMS
- net MTMS: now also J2.1 (Pin_1)
- net io47: no longer names the net of U1.24 (IO47)
- net io47: no longer R19.1
- net io48: no longer names the net of R22.1
- net io48: now also USBC1.B5 (CC2); no longer U1.25 (IO48)
- net io5 renamed GPIO5
- net GPIO5: now also U6.2
- net io6 renamed GPIO6
- net GPIO6: now also P1.3
- removed net io7: R7.1, TH1.2, U1.7 (IO7)
- net u0rxd renamed RXD
- net RXD: now also J1.3 (Pin_3)
- net u0txd renamed TXD
- net TXD: now also J1.2 (Pin_2)
- net usb+ renamed USB_D+
- net USB_D+: now also USBC1.A6 (DP1), USBC1.B6 (DP2)
- net usb- renamed USB_D-
- net USB_D-: now also USBC1.A7 (DN1), USBC1.B7 (DN2)
- new net: C10.1, C11.1, D6.2 (A), USBC1.A4 (VBUS), USBC1.A9 (VBUS), USBC1.B4 (VBUS), USBC1.B9 (VBUS)
- new net: R21.1, USBC1.A5 (CC1)
- new net: C7.1, U8.6 (BST)
- new net: F2.2, H1.1
- new net: BUZZER1.1 (+), R5.2
- new net: BUZZER1.2, R6.2
- new net: D1.2 (A), H10.1, Q1.3 (C), R6.1
- new net: H8.1, LED1.3 (DO)
- new net: D4.1 (K), U6.1
- new net: D2.1 (K), U5.1
- new net +5V: C6.1, D6.1 (K), F2.1, H6.1, U8.2 (EN), U8.3 (IN)
- new net GPIO10_SDA: J3.4 (Pin_4), R8.1, U1.18 (IO10)
- new net GPIO7: R13.1, TH1.1, U1.7 (IO7)
- no-connect marks 13 -> 17
Other:
- note added: "1-WIRE"
- note added: "BUZZER"
- note added: "CUSTOM INPUT"
- note added: "ESP32-S3-WROOM-1U-N16R2"
- note added: "I2C"
- note added: "JTAG"
- note added: "MDB"
- note added: "PCB MOUNTING HOLES"
- note added: "RELAY 1"
- note added: "RELAY 2"
- note added: "RGB LED"
- note added: "Thermistor"
- note added: "UART DEBUG"
- note added: "USB Type C"
- note added: "VOLTAGE REGULATOR INPUT: 3.8V to 32V"

Commit message: feat(wroom-1u): update PCB to rev1.3 (15A relay upgrade) and add fabrication gerbers
- Relay outputs redesigned: SRD-03VDC-SL-C 15A-class relays (K2/K3) driven
  low-side by MMBT3904 (Q2/Q3) with 1N4148WS flyback diodes, switched
  through TLP785 optocouplers (U4/U5) for GPIO isolation
- README rewritten to match rev1.3: updated reference designators, honest
  status section (4 minor ERC items, PCB/schematic re-sync pending),
  known relay drive-logic inversion documented as an open point
- Add gerber_to_order/ (JLCPCB, PCBWay) fabrication archives, versioned via
  .gitignore whitelist update

Note: PCB/schematic parity re-sync (reference renumbering from the relay
stage addition) and a voltage regulator issue are still open, handed off
to the hardware engineer for follow-up before ordering.
Parts:
- removed D3, D5: BAT760-7, Diode_SMD:D_SOD-323, symbol Device:D_Schottky
- removed H6: +5V, TestPoint:TestPoint_Pad_D1.0mm, symbol Mechanical:MountingHole_Pad
- removed H7: +3V3, TestPoint:TestPoint_Pad_D1.0mm, symbol Mechanical:MountingHole_Pad
- removed P1, P2, P3: WJ500V-5.08-3P-14-00A, Global Libraries:CONN-TH_3P-P5.00_WJ500V-5.08-3P_C72334, symbol globral_library:WJ500V-5.08-3P-14-00A
- removed P7, P8: WJ500V-5.08-2P-14-00A, Global Libraries:CONN-TH_2P-P5.00_WJ500V-5.08-2P_C8465, symbol globral_library:WJ500V-5.08-2P-14-00A
- removed R15: 1KΩ, Resistor_SMD:R_0603_1608Metric, symbol Device:R
- removed R4: 4.7KΩ, Resistor_SMD:R_0603_1608Metric, symbol Device:R
- removed R6: 0R, Resistor_SMD:R_0603_1608Metric_Pad0.98x0.95mm_HandSolder, symbol Device:R_Small
- added D4, D5: 1N4148WS, Diode_SMD:D_SOD-323, symbol Diode:1N4148WS
- added H11: Buzzer_IN, TestPoint:TestPoint_Pad_D1.0mm, symbol Mechanical:MountingHole_Pad
- added H12: Buzzer_OUT, TestPoint:TestPoint_Pad_D1.0mm, symbol Mechanical:MountingHole_Pad
- added K2, K3: SRD-03VDC-SL-C, Global Libraries:RELAY-TH_SRD-XXVDC-XL-C_C24585, symbol globral_library:SRD-03VDC-SL-C
- added P10, P11, P7, P8, P9: WJ500V-5.08-3P-14-00A, Global Libraries:CONN-TH_3P-P5.00_WJ500V-5.08-3P_C72334, symbol globral_library:WJ500V-5.08-3P-14-00A
- added R16: 0R, Resistor_SMD:R_0603_1608Metric_Pad0.98x0.95mm_HandSolder, symbol Device:R_Small
- added R23: 270Ω, Resistor_SMD:R_0603_1608Metric, symbol Device:R
- added R26, R28: 10KΩ, Resistor_SMD:R_0603_1608Metric, symbol Device:R
- added R27, R29: 100Ω, Resistor_SMD:R_0603_1608Metric, symbol Device:R
- added R6: 4.7KΩ, Resistor_SMD:R_0603_1608Metric, symbol Device:R
- added U4, U5: TLP785, Global Libraries:SMD-4_L4.6-W6.5-P2.54-LS10.2-BR_C45445, symbol Isolator:TLP785
- D2: LCSC C2128 -> (none); MFR.Part # 1N4148WS -> (none)
- D3: renamed from D4; LCSC C2128 -> (none); MFR.Part # 1N4148WS -> (none)
- F1: renamed from F2; footprint Capacitor_SMD:C_1812_4532Metric -> (none); LCSC C7542972 -> (none); MFR.Part # 1812L110/33GR -> (none)
- H1: renamed from H2; footprint MountingHole:MountingHole_2.7mm_M2.5_ISO7380 -> (none)
- H10: value Buzzer_OUT -> DO
- H2: renamed from H3; footprint MountingHole:MountingHole_2.7mm_M2.5_ISO7380 -> (none)
- H3: renamed from H4; footprint MountingHole:MountingHole_2.7mm_M2.5_ISO7380 -> (none)
- H4: renamed from H5; footprint MountingHole:MountingHole_2.7mm_M2.5_ISO7380 -> (none)
- H8: value DO -> +5V
- H9: value Buzzer_IN -> +3V3
- R12: footprint Resistor_SMD:R_0603_1608Metric -> (none); LCSC C23179 -> (none); MFR.Part # 0603WAF4700T5E -> (none)
- R14: footprint Resistor_SMD:R_0603_1608Metric -> (none); LCSC C14676 -> (none); MFR.Part # RC0603JR-071KL -> (none)
- R15: renamed from R16; footprint Resistor_SMD:R_0603_1608Metric -> (none); LCSC C23179 -> (none); MFR.Part # 0603WAF4700T5E -> (none)
- R19: value 1KΩ -> 270Ω; LCSC C14676 -> C22966; MFR.Part # RC0603JR-071KL -> 0603WAF2700T5E
- U2: renamed from U5; footprint Global Libraries:SMD-4_L4.6-W6.5-P2.54-LS10.2-BR_C45445 -> Package_DIP:DIP-4_W7.62mm; LCSC C45445 -> (none); MFR.Part # TLP785(GB-TP6,F -> (none)
- U3: renamed from U6; footprint Global Libraries:SMD-4_L4.6-W6.5-P2.54-LS10.2-BR_C45445 -> Package_DIP:DIP-4_W7.62mm; LCSC C45445 -> (none); MFR.Part # TLP785(GB-TP6,F -> (none)
- renumbered H1 to H7
Connections:
- net +3V3: now also D4.1 (K), D5.1 (K), H11.1, K2.1, K3.1, P7.2, P8.2, P9.2, R26.1, R28.1, R6.1
- net +5V: now also H8.1
- net GND: now also P7.1, P8.1, P9.1, U4.2, U4.3, U5.2, U5.3
- net GPIO1: now also R23.1; no longer R19.2
- net GPIO15: now also P7.3, P9.3, R6.2; no longer P4.3, P6.3
- net GPIO16: now also P8.3; no longer P5.3
- net GPIO17: now also P5.3
- net GPIO18: now also P6.3
- net GPIO2: now also R19.1
- net GPIO6: now also P4.3
- net at Q2.1 (B): now also R27.2
- net at Q2.3 (C): now also D4.2 (A), K2.4
- net at BUZZER1.2: now also R16.2
- net at D1.2 (A), Q1.3 (C): now also H12.1, R16.1; no longer H10.1
- net at LED1.3 (DO): now also H10.1; no longer H8.1
- net at Q3.3 (C): now also D5.2 (A), K3.4
- net at Q3.1 (B): now also R29.2; no longer R19.1
- new net: R23.2, U5.1
- new net: R26.2, R27.1, U5.4
- new net: R28.2, R29.1, U4.4
- new net: R19.2, U4.1
- new net: K3.2, P10.1
- new net: K3.5, P10.2
- new net: K3.3, P10.3
- new net: K2.2, P11.1
- new net: K2.5, P11.2
- new net: K2.3, P11.3
Other:
- note added: "ESP32 s3 Bootstraping pins GPIO0: Download / Flash mode select. GPIO3: JTAG / boot config related. GPIO45: Voltage / boot config strapping. GPIO46: Boot config strapping"
- note added: "JTAG Special pins MTCK GPIO39 MTDO GPIO40 MTDI GPIO41 MTMS GPIO42 JTAG PINS ARE MAINLY INPUT ONLY"
- note added: "Special Purpose pins for Internal Debugginh GPIO47 GPIO48"
- moved on the sheet: D2, D3, F1, H1, H2, H3, H4, H7, R12, R14, R15, U2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

Commit message: feat(wroom-1u): update PCB to rev1.4 (adjustable buck + schematic re-sync)
Swap U8 buck regulator from fixed-output AP63203QWU-7 to adjustable
AP63201WU-7, with a new external feedback divider (R23 196k / R24 62k)
and feed-forward cap (C19 100pF) to set the 3.3V rail.

Complete the schematic/PCB re-sync left open in rev1.3: the orphaned
1-Wire pull-up (R4) is now properly linked, and all connector/optocoupler
references have been renumbered and re-annotated consistently across
schematic and PCB (P1-P9, H1-H10, U3/U5/U6). Fix an accidental sheet
label ("mdb_slave_sharnobile" -> "mdb_slave_esp32s3-wroom-1u") picked up
during the KiCad resync. Regenerate gerbers for JLCPCB/PCBWay.

README updated to match: rev1.4, new buck part/feedback network, and all
renumbered connector references.
Parts:
- removed D4: 1N4148WS, Diode_SMD:D_SOD-323, symbol Diode:1N4148WS
- removed H11: Buzzer_IN, TestPoint:TestPoint_Pad_D1.0mm, symbol Mechanical:MountingHole_Pad
- removed H12: Buzzer_OUT, TestPoint:TestPoint_Pad_D1.0mm, symbol Mechanical:MountingHole_Pad
- removed P10, P11, P7: WJ500V-5.08-3P-14-00A, Global Libraries:CONN-TH_3P-P5.00_WJ500V-5.08-3P_C72334, symbol globral_library:WJ500V-5.08-3P-14-00A
- removed R16: 0R, Resistor_SMD:R_0603_1608Metric_Pad0.98x0.95mm_HandSolder, symbol Device:R_Small
- removed R6: 4.7KΩ, Resistor_SMD:R_0603_1608Metric, symbol Device:R
- removed U5: TLP785, Global Libraries:SMD-4_L4.6-W6.5-P2.54-LS10.2-BR_C45445, symbol Isolator:TLP785
- added C19: 100pF, Capacitor_SMD:C_0603_1608Metric, symbol Device:C
- added D3: 1N4148WS, Diode_SMD:D_SOD-323, symbol Diode:1N4148WS
- added H6: +5V, TestPoint:TestPoint_Pad_D1.0mm, symbol Mechanical:MountingHole_Pad
- added H7: +3V3, TestPoint:TestPoint_Pad_D1.0mm, symbol Mechanical:MountingHole_Pad
- added P1, P2, P3: WJ500V-5.08-3P-14-00A, Global Libraries:CONN-TH_3P-P5.00_WJ500V-5.08-3P_C72334, symbol globral_library:WJ500V-5.08-3P-14-00A
- added R15: 270Ω, Resistor_SMD:R_0603_1608Metric, symbol Device:R
- added R24: 62KΩ, Resistor_SMD:R_0603_1608Metric, symbol Device:R
- added R4: 4.7KΩ, Resistor_SMD:R_0603_1608Metric, symbol Device:R
- added R6: 0R, Resistor_SMD:R_0603_1608Metric_Pad0.98x0.95mm_HandSolder, symbol Device:R_Small
- added U3: TLP785, Global Libraries:SMD-4_L4.6-W6.5-P2.54-LS10.2-BR_C45445, symbol Isolator:TLP785
- D2: LCSC (none) -> C2128; MFR.Part # (none) -> 1N4148WS
- D4: renamed from D3; LCSC (none) -> C2128; MFR.Part # (none) -> 1N4148WS
- F2: renamed from F1; footprint (none) -> Capacitor_SMD:C_1812_4532Metric; LCSC (none) -> C7542972; MFR.Part # (none) -> 1812L110/33GR
- H10: value DO -> Buzzer_OUT
- H2: renamed from H1; footprint (none) -> MountingHole:MountingHole_2.7mm_M2.5_ISO7380
- H3: renamed from H2; footprint (none) -> MountingHole:MountingHole_2.7mm_M2.5_ISO7380
- H4: renamed from H3; footprint (none) -> MountingHole:MountingHole_2.7mm_M2.5_ISO7380
- H5: renamed from H4; footprint (none) -> MountingHole:MountingHole_2.7mm_M2.5_ISO7380
- H8: value +5V -> DO
- H9: value +3V3 -> Buzzer_IN
- K2, K3: LCSC (none) -> C24585; MFR.Part # (none) -> SRD-03VDC-SL-C; Manufacturer Part SRD-03VDC-SL-C -> (none); Supplier LCSC -> (none); Supplier Part C24585 -> (none)
- L1: LCSC C12589 -> C75929; MFR.Part # SDFL1608Q3R3KTF -> SDFL1608S6R8KTF
- R12: footprint (none) -> Resistor_SMD:R_0603_1608Metric; LCSC (none) -> C23179; MFR.Part # (none) -> 0603WAF4700T5E
- R14: footprint (none) -> Resistor_SMD:R_0603_1608Metric; LCSC (none) -> C14676; MFR.Part # (none) -> RC0603JR-071KL
- R16: renamed from R15; footprint (none) -> Resistor_SMD:R_0603_1608Metric; LCSC (none) -> C23179; MFR.Part # (none) -> 0603WAF4700T5E
- R23: value 270Ω -> 196KΩ; LCSC C22966 -> C22930; MFR.Part # 0603WAF2700T5E -> 0603WAF1963T5E
- U5: renamed from U2; footprint Package_DIP:DIP-4_W7.62mm -> Global Libraries:SMD-4_L4.6-W6.5-P2.54-LS10.2-BR_C45445; LCSC (none) -> C45445; MFR.Part # (none) -> TLP785(GB-TP6,F
- U6: renamed from U3; footprint Package_DIP:DIP-4_W7.62mm -> Global Libraries:SMD-4_L4.6-W6.5-P2.54-LS10.2-BR_C45445; LCSC (none) -> C45445; MFR.Part # (none) -> TLP785(GB-TP6,F
- U8: value AP63203QWU-7 -> AP63201WU-7; LCSC C5248536 -> C2071044; MFR.Part # AP63203QWU-7 -> AP63201WU-7
- renumbered H7 to H1
Connections:
- net +3V3: now also R23.1, C19.1, D3.1 (K), H7.1, P1.2, P2.2, P3.2, R4.1; no longer P8.2, P9.2, U8.1 (FB)
- net +5V: now also H6.1; no longer H8.1
- net GND: now also P1.1, P2.1, P3.1, R24.2, U3.2, U3.3; no longer P8.1, P9.1
- net GPIO1: now also R15.1; no longer R23.1
- net GPIO15: now also P4.3, P6.3, R4.2; no longer P9.3
- net GPIO16: now also P5.3; no longer P8.3
- net GPIO17: now also P2.3; no longer P5.3
- net GPIO18: now also P3.3; no longer P6.3
- net GPIO6: now also P1.3; no longer P4.3
- net at D1.2 (A), Q1.3 (C): now also H10.1, R6.1
- net at K2.4, Q2.3 (C): now also D3.2 (A)
- net at R23.2: now also U8.1 (FB), C19.2, R24.1
- net at R26.2, R27.1: now also U3.4
- net at LED1.3 (DO): now also H8.1; no longer H10.1
- net at BUZZER1.2: now also R6.2
- net at K3.2: now also P9.1
- net at K3.5: now also P9.2
- net at K3.3: now also P9.3
- net at K2.2: now also P8.1
- net at K2.5: now also P8.2
- net at K2.3: now also P8.3
- new net: R15.2, U3.1
Other:
- note added: "Special Purpose pins for Internal Debugging GPIO47 GPIO48"
- note removed: "Special Purpose pins for Internal Debugginh GPIO47 GPIO48"
- moved on the sheet: D2, D4, F2, H1, H2, H3, H4, H5, R12, R14, R16, U5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
