File: kicad/mdb_slave_esp32s3-wroom-1u/mdb_slave_esp32s3-wroom-1u.kicad_sch (KiCad schematic)
At the start: 87 parts, among them J1 Conn_01x06_Pin, J2 Conn_01x06_Pin, J3 Conn_01x04_Pin, K2 SRD-03VDC-SL-C, K3 SRD-03VDC-SL-C, P1 WJ500V-5.08-3P-14-00A, P2 WJ500V-5.08-3P-14-00A, P3 WJ500V-5.08-3P-14-00A, P4 WJ500V-5.08-3P-14-00A, P5 WJ500V-5.08-3P-14-00A, P6 WJ500V-5.08-3P-14-00A, P8 WJ500V-5.08-3P-14-00A, P9 WJ500V-5.08-3P-14-00A, Q1 MMBT3904, Q2 MMBT3904, Q3 MMBT3904, U1 ESP32-S3-WROOM-1U-N16R2, U3 TLP785, U4 TLP785, U5 TLP785, U6 TLP785, U8 AP63201WU-7

Commit message: fix(wroom-1u): change R26/R28 to 1KΩ (rev1.4.1)
R26 and R28 changed from 10KΩ (LCSC C25804) to 1KΩ (LCSC C14676) in
schematic and PCB, silkscreen bumped to REV 1.4.1, gerbers
regenerated, README revision/status synced.

Co-Authored-By: Claude Sonnet 5 <noreply@anthropic.com>
Parts:
- R26, R28: value 10KΩ -> 1KΩ; LCSC C25804 -> C14676; MFR.Part # 0603WAF1002T5E -> RC0603JR-071KL
Other:
- note added: "Rev. 1.4.1"
- moved on the sheet: P4, P5, P6, R11, R4, R7
