File: kicad/mdb_slave_esp32s3-wroom-1u/mdb_slave_esp32s3-wroom-1u.kicad_pcb (KiCad board)
At the start: 4 copper layers, 149.8 x 38.5 mm, 88 parts, among them J1 Conn_01x06_Pin, J2 Conn_01x06_Pin, J3 Conn_01x04_Pin, K2 SRD-03VDC-SL-C, K3 SRD-03VDC-SL-C, P1 WJ500V-5.08-3P-14-00A, P2 WJ500V-5.08-3P-14-00A, P3 WJ500V-5.08-3P-14-00A, P4 WJ500V-5.08-3P-14-00A, P5 WJ500V-5.08-3P-14-00A, P6 WJ500V-5.08-3P-14-00A, P8 WJ500V-5.08-3P-14-00A, P9 WJ500V-5.08-3P-14-00A, Q1 MMBT3904, Q2 MMBT3904, Q3 MMBT3904, U1 ESP32-S3-WROOM-1U-N16R2, U3 TLP785, U4 TLP785, U5 TLP785, U6 TLP785, U8 AP63201WU-7

Commit message: fix(wroom-1u): change R26/R28 to 1KΩ (rev1.4.1)
R26 and R28 changed from 10KΩ (LCSC C25804) to 1KΩ (LCSC C14676) in
schematic and PCB, silkscreen bumped to REV 1.4.1, gerbers
regenerated, README revision/status synced.

Co-Authored-By: Claude Sonnet 5 <noreply@anthropic.com>
Parts:
- R26, R28: value 10KΩ -> 1KΩ
Other:
- board text added: "REV 1.4.1"
- board text removed: "REV 1.4"
Changed lines of the file:
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@@
 			)
 		)
-		(property "Value" "10KΩ"
+		(property "Value" "1KΩ"
 			(at 0 1.43 0)
 			(layer "F.Fab")
@@
 			)
 		)
-		(property "Description" "100mW Thick Film Resistors 75V ±100ppm/℃ ±1% 1kΩ 0603 Chip Resistor - Surface Mount ROHS"
+		(property "Description" "100mW Thick Film Resistors 75V ±100ppm/℃ ±1% 1kΩ 0603 Chip Resistor - Surface Mount ROHS "
 			(at 0 0 0)
 			(layer "F.Fab")
@@
 			)
 		)
-		(property "MFR.Part #" "0603WAF1002T5E"
+		(property "MFR.Part #" "RC0603JR-071KL "
 			(at 0 0 180)
 			(unlocked yes)
@@
 			)
 		)
-		(property "LCSC" "C25804"
+		(property "LCSC" "C14676"
 			(at 0 0 180)
 			(unlocked yes)
@@
 			)
 		)
-		(property "Value" "10KΩ"
+		(property "Value" "1KΩ"
 			(at 0 1.43 90)
 			(layer "F.Fab")
@@
 			)
 		)
-		(property "Description" "100mW Thick Film Resistors 75V ±100ppm/℃ ±1% 1kΩ 0603 Chip Resistor - Surface Mount ROHS"
+		(property "Description" "100mW Thick Film Resistors 75V ±100ppm/℃ ±1% 1kΩ 0603 Chip Resistor - Surface Mount ROHS "
 			(at 0 0 90)
 			(layer "F.Fab")
@@
 			)
 		)
-		(property "MFR.Part #" "0603WAF1002T5E"
+		(property "MFR.Part #" "RC0603JR-071KL"
 			(at 0 0 90)
 			(unlocked yes)
@@
 			)
 		)
-		(property "LCSC" "C25804"
+		(property "LCSC" "C14676"
 			(at 0 0 90)
 			(unlocked yes)
@@
 		)
 	)
-	(gr_text "REV 1.4"
-		(at 70.75 126.25 180)
+	(gr_text "REV 1.4.1"
+		(at 69.5 126.25 180)
 		(layer "B.SilkS")
 		(effects
